File: parasite-2/parasite.kicad_pcb (KiCad board)
At the start: 2 copper layers, 30 x 118.2 mm, 32 parts, among them J1 Conn_01x02_Female, J2 Conn_01x01, J3 Conn_01x01, Q1 MMBT3904, Q2 MMBT3904, SW1 SW_Push, SW2 SW_Push, U1 XB3303A

Commit message: update
Parts:
- removed 3V3, GND: Conn_01x01, pin:PinHeader_1x01_P2.54mm_Vertical
- J2, J3: value Conn_01x01 -> Conn_01x02; footprint pin:PinHeader_1x01_P2.54mm_Vertical -> Connector_PinHeader_2.54mm:PinHeader_1x02_P2.54mm_Vertical
- moved J3 30.2 mm to (130.3, 84.3), turned to 180 degrees
- moved J2 0.99 mm to (130.8, 51.4), turned to 0 degrees
Connections:
- J3 pad 1: /RX -> +BATT
- MOD1 pad 15: (no net) -> GND
- MOD1 pad 38: (no net) -> GND
Routing:
- net GND: track 175.2 -> 242.7 mm, vias 12 -> 16
- net /en: track 40.3 -> 21.4 mm, vias 3 -> 2
- net +3V3: track 63.5 -> 55.5 mm
- net +BATT: track 90.1 -> 93.7 mm
- net /TX: track 6.27 -> 5.19 mm
